Commit message: updated the urdf to work again

File: urdf/spotmicroai.urdf.xacro (robot description, xacro)
@@ -178,5 +178,5 @@
       <visual>
         <geometry>
-        <mesh filename="../STL/files/foot.stl" scale="0.001 0.001 0.001"/>
+        <mesh filename="../Hardware/other/foot.stl" scale="0.001 0.001 0.001"/>
         </geometry>
         <origin rpy="0 -0.40010 0" xyz="0 -0.01 0"/>
